File: Eagle Boards/CableBotEndEffector/EndEffector.brd (EAGLE design)
At the start: 38.1 x 38.1 mm, 14 parts

Commit message: xbee board update
Parts:
- R1: value 100k -> 10k
Changed lines of the file:
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@@
 <attribute name="VALUE" x="29.845" y="5.715" size="1.27" layer="27" rot="R90"/>
 </element>
-<element name="R1" library="CabelBot" package="_0603" value="100k" x="25.4" y="4.318" smashed="yes">
+<element name="R1" library="CabelBot" package="_0603" value="10k" x="25.4" y="4.318" smashed="yes">
 <attribute name="NAME" x="23.5585" y="3.683" size="0.8128" layer="25" ratio="18" rot="R90"/>
 <attribute name="VALUE" x="24.511" y="5.2387" size="0.4064" layer="27" ratio="10"/>
