File: Eagle Boards/CableBotEndEffector/Tiva_Xbee.brd (EAGLE design)
At the start: 17.8 x 25.4 mm, 5 parts

Commit message: xbee board update
Parts:
- R1: value (none) -> 10k
Changed lines of the file:
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@@
 <attribute name="VALUE" x="11.176" y="3.937" size="0.6096" layer="27" font="vector" ratio="20" rot="R180"/>
 </element>
-<element name="R1" library="CabelBot" package="_0603" value="" x="15.24" y="2.54" smashed="yes" rot="R90">
+<element name="R1" library="CabelBot" package="_0603" value="10k" x="15.24" y="2.54" smashed="yes" rot="R90">
 <attribute name="NAME" x="14.2875" y="1.27" size="0.8128" layer="25" ratio="18" rot="R90"/>
 <attribute name="VALUE" x="16.7323" y="1.27" size="0.4064" layer="27" ratio="10" rot="R90"/>

Commit message: clean up boards
Parts:
- added J2: (no value), SparkFun-Connectors:1X05
- moved J1 1.65 mm to (11.4, 2.54)
Routing:
- net DIO2: track 20.7 -> 19.6 mm
- net GND: track 34.1 -> 34.8 mm
Other:
- board size 17.8 x 25.4 mm -> 17.8 x 30.5 mm
Changed lines of the file:
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@@
 <?xml version="1.0" encoding="utf-8"?>
 <!DOCTYPE eagle SYSTEM "eagle.dtd">
-<eagle version="9.4.0">
+<eagle version="9.2.2">
 <drawing>
 <settings>
@@
 <board>
 <plain>
-<wire x1="0" y1="22.86" x2="0" y2="2.54" width="0" layer="20"/>
+<wire x1="0" y1="27.94" x2="0" y2="2.54" width="0" layer="20"/>
 <wire x1="0" y1="2.54" x2="2.54" y2="0" width="0" layer="20" curve="90"/>
 <wire x1="2.54" y1="0" x2="15.24" y2="0" width="0" layer="20"/>
 <wire x1="15.24" y1="0" x2="17.78" y2="2.54" width="0" layer="20" curve="90"/>
-<wire x1="17.78" y1="2.54" x2="17.78" y2="22.86" width="0" layer="20"/>
-<wire x1="17.78" y1="22.86" x2="15.24" y2="25.4" width="0" layer="20" curve="90"/>
-<wire x1="15.24" y1="25.4" x2="2.54" y2="25.4" width="0" layer="20"/>
-<wire x1="2.54" y1="25.4" x2="0" y2="22.86" width="0" layer="20" curve="90"/>
+<wire x1="17.78" y1="2.54" x2="17.78" y2="26.67" width="0" layer="20"/>
+<wire x1="17.78" y1="26.67" x2="15.24" y2="30.48" width="0" layer="20" curve="90"/>
+<wire x1="15.24" y1="30.48" x2="2.54" y2="30.48" width="0" layer="20"/>
+<wire x1="2.54" y1="30.48" x2="0" y2="27.94" width="0" layer="20" curve="90"/>
 <text x="3.937" y="3.556" size="0.635" layer="21">GND    3V3    DIO</text>
 </plain>
@@
 <attribute name="VALUE" x="7.2707" y="17.526" size="0.4064" layer="28" ratio="10" rot="MR90"/>
 </element>
-<element name="J1" library="CabelBot" package="1X03" package3d_urn="urn:adsk.eagle:package:38063/1" value="" x="9.906" y="1.905" smashed="yes" rot="R180">
-<attribute name="VALUE" x="11.176" y="3.937" size="0.6096" layer="27" font="vector" ratio="20" rot="R180"/>
+<element name="J1" library="CabelBot" package="1X03" package3d_urn="urn:adsk.eagle:package:38063/1" value="" x="11.43" y="2.54" smashed="yes" rot="R180">
+<attribute name="VALUE" x="12.7" y="4.572" size="0.6096" layer="27" font="vector" ratio="20" rot="R180"/>
 </element>
 <element name="R1" library="CabelBot" package="_0603" value="10k" x="15.24" y="2.54" smashed="yes" rot="R90">
@@
 </element>
 <element name="U$1" library="CabelBot" package="XBEE3_MICRO" value="XBEE3_DIO" x="8.89" y="15.24" smashed="yes"/>
+<element name="J2" library="SparkFun-Connectors" library_urn="urn:adsk.eagle:library:513" package="1X05" package3d_urn="urn:adsk.eagle:package:38104/1" value="" x="3.81" y="27.94" smashed="yes">
+<attribute name="NAME" x="2.54" y="29.337" size="0.6096" layer="25" font="vector" ratio="20"/>
+<attribute name="VALUE" x="2.54" y="25.908" size="0.6096" layer="27" font="vector" ratio="20"/>
+</element>
 </elements>
 <signals>
@@
 <wire x1="14.83546875" y1="20.59938125" x2="15.184121875" y2="20.59938125" width="0.254" layer="1"/>
 <wire x1="15.184121875" y1="20.59938125" x2="15.6718" y2="21.087059375" width="0.254" layer="1"/>
-<wire x1="4.826" y1="1.905" x2="4.826" y2="3.73566875" width="0.254" layer="1"/>
-<wire x1="4.826" y1="3.73566875" x2="3.81" y2="4.75166875" width="0.254" layer="1"/>
-<wire x1="3.81" y1="4.75166875" x2="3.81" y2="9.5739125" width="0.254" layer="1"/>
+<wire x1="3.81" y1="3.81" x2="3.81" y2="9.5739125" width="0.254" layer="1"/>
+<wire x1="6.35" y1="2.54" x2="5.08" y2="2.54" width="0.254" layer="1"/>
+<wire x1="5.08" y1="2.54" x2="3.81" y2="3.81" width="0.254" layer="1"/>
 <wire x1="3.81" y1="9.5739125" x2="14.83546875" y2="20.59938125" width="0.254" layer="1"/>
 <wire x1="5.334" y1="17.907" x2="5.461" y2="18.034" width="0.254" layer="16"/>
@@
 <contactref element="J1" pad="1"/>
 <contactref element="R1" pad="2"/>
-<wire x1="9.906" y1="1.905" x2="15.24" y2="3.302" width="0.254" layer="1"/>
+<wire x1="15.24" y1="3.302" x2="14.478" y2="2.54" width="0.254" layer="1"/>
+<wire x1="14.478" y1="2.54" x2="11.43" y2="2.54" width="0.254" layer="1"/>
 <wire x1="16.50813125" y1="16.85034375" x2="16.9545" y2="16.403975" width="0.254" layer="1"/>
 <wire x1="15.6718" y1="17.338025" x2="16.15948125" y2="16.85034375" width="0.254" layer="1"/>
 <wire x1="16.15948125" y1="16.85034375" x2="16.50813125" y2="16.85034375" width="0.254" layer="1"/>
-<wire x1="16.9545" y1="16.403975" x2="16.9545" y2="7.02496875" width="0.254" layer="1"/>
-<wire x1="16.9545" y1="7.02496875" x2="16.51" y2="6.58046875" width="0.254" layer="1"/>
-<wire x1="16.51" y1="6.58046875" x2="16.51" y2="6.35" width="0.254" layer="1"/>
-<wire x1="16.51" y1="6.35" x2="15.24" y2="3.302" width="0.254" layer="1"/>
+<wire x1="16.9545" y1="16.403975" x2="16.9545" y2="5.0165" width="0.254" layer="1"/>
+<wire x1="16.9545" y1="5.0165" x2="15.24" y2="3.302" width="0.254" layer="1"/>
 </signal>
 <signal name="DIN">
@@
 which will not be processed correctly with this version.
 </note>
+<note version="8.2" severity="warning">
+Since Version 8.2, EAGLE supports online libraries. The ids
+of those online libraries will not be understood (or retained)
+with this version.
+</note>
 <note version="8.3" severity="warning">
