File: Eagle Boards/CableBotEndEffector/Tiva_Xbee.sch (EAGLE design)
At the start: 5 parts

Commit message: xbee board update
Parts:
- R1: value (none) -> 10k
Changed lines of the file:
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@@
 <part name="U$2" library="CabelBot" deviceset="GND" device=""/>
 <part name="U$3" library="CabelBot" deviceset="3.3V" device=""/>
-<part name="R1" library="CabelBot" deviceset="RESISTOR" device="_0603"/>
+<part name="R1" library="CabelBot" deviceset="RESISTOR" device="_0603" value="10k"/>
 <part name="U$4" library="CabelBot" deviceset="GND" device=""/>
 </parts>

Commit message: clean up boards
Parts:
- added J2: (no value), SparkFun-Connectors:CONN_05
Changed lines of the file:
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@@
 <?xml version="1.0" encoding="utf-8"?>
 <!DOCTYPE eagle SYSTEM "eagle.dtd">
-<eagle version="9.4.0">
+<eagle version="9.2.2">
 <drawing>
 <settings>
@@
 <part name="R1" library="CabelBot" deviceset="RESISTOR" device="_0603" value="10k"/>
 <part name="U$4" library="CabelBot" deviceset="GND" device=""/>
+<part name="J2" library="SparkFun-Connectors" library_urn="urn:adsk.eagle:library:513" deviceset="CONN_05" device="" package3d_urn="urn:adsk.eagle:package:38104/1"/>
 </parts>
 <sheets>
@@
 <instance part="U$4" gate="G$1" x="50.8" y="43.18" smashed="yes">
 <attribute name="VALUE" x="49.276" y="40.64" size="1.27" layer="96"/>
+</instance>
+<instance part="J2" gate="G$1" x="78.74" y="66.04" smashed="yes">
+<attribute name="VALUE" x="76.2" y="56.134" size="1.778" layer="96" font="vector"/>
+<attribute name="NAME" x="76.2" y="74.168" size="1.778" layer="95" font="vector"/>
 </instance>
 </instances>
@@
 which will not be processed correctly with this version.
 </note>
+<note version="8.2" severity="warning">
+Since Version 8.2, EAGLE supports online libraries. The ids
+of those online libraries will not be understood (or retained)
+with this version.
+</note>
 <note version="8.3" severity="warning">
