File: Eagle Boards/Main Board/main.sch (EAGLE design)
At the start: 30 parts, among them IC1 REG1117, IC2 FT232RL-TUBE, J3 PROG, J4 PROG_RST, U1 TM4C123GH6PMIPM64-L, Y1 ABM3-16.000MHZ-B2-T

Commit message: finish most of board design prelim
Parts:
- removed TEST: MOM_SWITCH, tiva:MOM_SWITCH
- added AROW, BROW, CROW, DROW, EROW, FROW: (no value), SparkFun-Connectors:CONN_08"
- added B1: (no value), tiva:B3S-1000
- added C18, C19: 1uF, adafruit:C-USC0805
- added CR1, CR2, CR3: ST26C31BTR, tiva:ST26C31BTR
- added IC3: REG1117, burr-brown:REG1117
- added J7: (no value), SparkFun-Connectors:CONN_02
- added MOTOR1, MOTOR2, MOTOR3, MOTOR4: (no value), SparkFun-Connectors:CONN_06NO_SILK_FEMALE_PTH
- added R10, R11, R12, R13, R14, R15, R16, R17, R18, R19, R20, R21, R22, R23, R24, R25, R26, R27, R28, R5, R6, R7, R8, R9: 10k, adafruit:R-US_R0603
- added U10, U11, U12, U13, U14, U3, U4, U5, U6, U7, U8, U9: BSS138SOT-23-3L-L, tiva:BSS138SOT-23-3L-L
- R1: device adafruit:R-US_R0805 -> adafruit:R-US_R0603
Connections:
- removed net OSC2: C4.1, Y1.2
- new net !DIR1: CR3.!AOUT, MOTOR1.6
- new net !DIR2: CR3.!BOUT, MOTOR2.6
- new net !DIR3: CR3.!COUT, MOTOR3.6
- new net !DIR4: CR3.!DOUT, MOTOR4.6
- new net !EN1: CR2.!AOUT, MOTOR1.4
- new net !EN2: CR2.!BOUT, MOTOR2.4
- new net !EN3: CR2.!COUT, MOTOR3.4
- new net !EN4: CR2.!DOUT, MOTOR4.4
- new net !M1: CR1.!AOUT, MOTOR1.2
- new net !M2: CR1.!BOUT, MOTOR2.2
- new net !M3: CR1.!COUT, MOTOR3.2
- new net !M4: CR1.!DOUT, MOTOR4.2
- new net DIR1: CR3.AOUT, MOTOR1.5
- new net DIR1_SIG: CR3.AIN, R22.1, U11.D
- new net DIR2: CR3.BOUT, MOTOR2.5
- new net DIR2_SIG: CR3.BIN, R24.1, U12.D
- new net DIR3: CR3.COUT, MOTOR3.5
- new net DIR3_SIG: CR3.CIN, R26.1, U13.D
- new net DIR4: CR3.DOUT, MOTOR4.5
- new net DIR4_SIG: CR3.DIN, R28.1, U14.D
- new net EN1: CR2.AOUT, MOTOR1.3
- new net EN1_SIG: CR2.AIN, R14.1, U7.D
- new net EN2: CR2.BOUT, MOTOR2.3
- new net EN2_SIG: CR2.BIN, R16.1, U8.D
- new net EN3: CR2.COUT, MOTOR3.3
- new net EN3_SIG: CR2.CIN, R18.1, U9.D
- new net EN4: CR2.DOUT, MOTOR4.3
- new net EN4_SIG: CR2.DIN, R20.1, U10.D
- new net M1: CR1.AOUT, MOTOR1.1
- new net M1_SIG: CR1.AIN, R6.1, U3.D
- new net M2: CR1.BOUT, MOTOR2.1
- new net M2_SIG: CR1.BIN, R8.1, U4.D
- new net M3: CR1.COUT, MOTOR3.1
- new net M3_SIG: CR1.CIN, R10.1, U5.D
- new net M4: CR1.DOUT, MOTOR4.1
- new net M4_SIG: CR1.DIN, R12.1, U6.D
- new net N$36: FROW.1
- new net N$37: FROW.2
- new net N$38: FROW.3
- new net N$44: EROW.1
- new net N$45: EROW.2
- new net PA2: AROW.6, U1.PA2/SSI0CLK
- new net PA3: AROW.5, U1.PA3/SSI0FSS
- new net PA4: AROW.4, U1.PA4/SSI0RX
- new net PA5: AROW.3, U1.PA5/SSI0TX
- new net PA6: AROW.2, U1.PA6
- new net PA7: AROW.1, U1.PA7
- new net PB2: BROW.6, U1.PB2/I2C0SCL
- new net PB3: BROW.5, U1.PB3/I2C0SDA
- new net PB4: BROW.4, U1.PB4
- new net PB5: BROW.3, U1.PB5
- new net PC4: CROW.4, U1.PC4
- new net PC5: CROW.3, U1.PC5
- new net PC6: CROW.2, U1.PC6
- new net PC7: CROW.1, U1.PC7
- new net PD4: DROW.4, U1.PD4
- new net PD5: DROW.3, U1.PD5
- new net PE4: EROW.4, U1.PE4
- new net PE5: EROW.3, U1.PE5
- new net PF0: FROW.8, U1.PF0
- new net PF1: FROW.7, U1.PF1
- new net PF4: FROW.4, U1.PF4
- new net V_USB: IC2.VCC, S1.3, S1.6, U$1.VCC
- net !RST: now also B1.PD2; no longer TEST.PD2
- net 3.3V: now also J7.2, R11.2, R13.2, R15.2, R17.2, R19.2, R21.2, R23.2, R25.2, R27.2, R5.2, R7.2, R9.2, U10.G, U11.G, U12.G, U13.G, U14.G, U3.G, U4.G, U5.G, U6.G, U7.G, U8.G, U9.G
- net 5V: now also C19.1, CR1.VCC, CR2.VCC, CR3.VCC, IC3.VOUT, R10.2, R12.2, R14.2, R16.2, R18.2, R20.2, R22.2, R24.2, R26.2, R28.2, R6.2, R8.2; no longer IC2.VCC, S1.3, S1.6, U$1.VCC
- net GND: now also B1.PD1, C18.2, C19.2, C3.2, C4.2, CR1.!EN, CR1.EN, CR1.GND, CR2.!EN, CR2.EN, CR2.GND, CR3.!EN, CR3.EN, CR3.GND, IC3.GND, J7.1; no longer TEST.PD1
- net M_DIR_0: now also DROW.8, R21.1, U11.S
- net M_DIR_1: now also DROW.7, R23.1, U12.S
- net M_DIR_2: now also DROW.6, R25.1, U13.S
- net M_DIR_3: now also DROW.5, R27.1, U14.S
- net M_EN_0: now also EROW.8, R13.1, U7.S
- net M_EN_1: now also EROW.7, R15.1, U8.S
- net M_EN_2: now also EROW.6, R17.1, U9.S
- net M_EN_3: now also EROW.5, R19.1, U10.S
- net OSC0: now also C4.1, Y1.2
- net T0PWM0: now also BROW.2, R5.1, U3.S
- net T0PWM1: now also BROW.1, R7.1, U4.S
- net T1PWM0: now also FROW.6, R9.1, U5.S
- net T1PWM1: now also FROW.5, R11.1, U6.S
- net TCK: now also CROW.8
- net TDI: now also CROW.6
- net TDO: now also CROW.5
- net TMS: now also CROW.7
- net U0RX: now also AROW.8
- net U0TX: now also AROW.7
- net U1RX: now also BROW.8
- net U1TX: now also BROW.7
- net U2RX: now also DROW.2
- net U2TX: now also DROW.1
- net VBUS: now also C18.1, IC3.VIN
Other:
- note added: "5V Linear Regulator"
- note added: "check this part"

Commit message: fix a few chips. add RS485 Hookup
Parts:
- added J1: (no value), SparkFun-Connectors:CONN_02
- added R29, R4: 1.2k, resistor:R-US_R0805
- added R3: 100, resistor:R-US_R0805
- added RS485OUT: (no value), SparkFun-Connectors:CONN_05
- added U2: SN75LBC179D, tiva:SN75LBC179D
Connections:
- removed net VBUS: C16.1, C18.1, IC1.VIN, IC3.VIN, S1.2, S1.5
- new net !RS_RX: RS485OUT.4, U2.B
- new net !RS_TX: R29.1, R3.1, RS485OUT.2, U2.Z
- new net 5VIN: C19.1, IC3.VOUT, S1.1, S1.4
- new net RS_RX: RS485OUT.5, U2.A
- new net RS_TX: R3.2, R4.1, RS485OUT.3, U2.Y
- net 12V: now also C18.1, IC3.VIN; no longer S1.1, S1.4
- net 5V: now also C16.1, IC1.VIN, J1.2, R4.2, S1.2, S1.5, U2.VCC; no longer C14.1, C15.1, C19.1, IC3.VOUT
- net GND: now also J1.1, R29.2, RS485OUT.1, U2.GND
- net U2RX: now also U2.R
- net U2TX: now also U2.D
- net V_USB: now also C14.1, C15.1

Commit message: Update eagle files
Parts:
- renumbered U$1 to USB
Changed lines of the file:
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@@
 </part>
 <part name="GND10" library="SparkFun-PowerSymbols" library_urn="urn:adsk.eagle:library:530" deviceset="GND" device=""/>
-<part name="U$1" library="ZX62-AB-5PA_11_" deviceset="ZX62MICROUSB" device=""/>
+<part name="USB" library="ZX62-AB-5PA_11_" deviceset="ZX62MICROUSB" device=""/>
 <part name="GND11" library="SparkFun-PowerSymbols" library_urn="urn:adsk.eagle:library:530" deviceset="GND" device=""/>
 <part name="C13" library="adafruit" library_urn="urn:adsk.eagle:library:420" deviceset="C-US" device="C0805" package3d_urn="urn:adsk.eagle:package:6240337/1" value="0.1uF"/>
@@
 <attribute name="VALUE" x="58.42" y="68.326" size="1.778" layer="96" align="top-center"/>
 </instance>
-<instance part="U$1" gate="G$1" x="25.4" y="134.62" smashed="yes">
+<instance part="USB" gate="G$1" x="25.4" y="134.62" smashed="yes">
 <attribute name="NAME" x="29.21341875" y="132.07771875" size="1.7796" layer="95"/>
 </instance>
@@
 </segment>
 <segment>
-<pinref part="U$1" gate="G$1" pin="D+"/>
+<pinref part="USB" gate="G$1" pin="D+"/>
 <wire x1="20.32" y1="132.08" x2="20.32" y2="127" width="0.1524" layer="91"/>
 <label x="20.32" y="127" size="1.778" layer="95" rot="R90"/>
@@
 </segment>
 <segment>
-<pinref part="U$1" gate="G$1" pin="D-"/>
+<pinref part="USB" gate="G$1" pin="D-"/>
 <wire x1="22.86" y1="132.08" x2="22.86" y2="127" width="0.1524" layer="91"/>
 <label x="22.86" y="127" size="1.778" layer="95" rot="R90"/>
@@
 </segment>
 <segment>
-<pinref part="U$1" gate="G$1" pin="GND"/>
+<pinref part="USB" gate="G$1" pin="GND"/>
 <wire x1="17.78" y1="132.08" x2="17.78" y2="127" width="0.1524" layer="91"/>
 <pinref part="GND11" gate="1" pin="GND"/>
@@
 <net name="V_USB" class="0">
 <segment>
-<pinref part="U$1" gate="G$1" pin="VCC"/>
+<pinref part="USB" gate="G$1" pin="VCC"/>
 <wire x1="25.4" y1="132.08" x2="25.4" y2="127" width="0.1524" layer="91"/>
 <pinref part="SUPPLY3" gate="G$1" pin="V_USB"/>

Commit message: clean up boards
Parts:
- removed AROW, BROW, CROW, DROW, EROW, FROW: (no value), SparkFun-Connectors:CONN_08"
- removed C18, C19: 1uF, adafruit:C-USC0805
- removed CR2: ST26C31BTR, tiva:ST26C31BTR
- removed IC3: REG1117, burr-brown:REG1117
- removed R13, R14, R15, R16, R17, R18, R19, R20: 10k, adafruit:R-US_R0603
- removed RS485OUT: (no value), SparkFun-Connectors:CONN_05
- removed U10, U7, U8, U9: BSS138SOT-23-3L-L, tiva:BSS138SOT-23-3L-L
- added PROG, RS485: BM05B-ZESS, tiva:BM05B-ZESS
- 3.3V: value REG1117 -> 3.3VREG
- MOTOR1, MOTOR2, MOTOR3, MOTOR4: value (none) -> BM05B-ZESS; device SparkFun-Connectors:CONN_06NO_SILK_FEMALE_PTH -> tiva:BM05B-ZESS
- renumbered IC1 to 3.3V
Connections:
- removed net !EN1: CR2.!AOUT, MOTOR1.4
- removed net !EN2: CR2.!BOUT, MOTOR2.4
- removed net !EN3: CR2.!COUT, MOTOR3.4
- removed net !EN4: CR2.!DOUT, MOTOR4.4
- removed net 12V: C18.1, IC3.VIN
- removed net 5VIN: C19.1, IC3.VOUT, S1.1, S1.4
- removed net EN1: CR2.AOUT, MOTOR1.3
- removed net EN1_SIG: CR2.AIN, R14.1, U7.D
- removed net EN2: CR2.BOUT, MOTOR2.3
- removed net EN2_SIG: CR2.BIN, R16.1, U8.D
- removed net EN3: CR2.COUT, MOTOR3.3
- removed net EN3_SIG: CR2.CIN, R18.1, U9.D
- removed net EN4: CR2.DOUT, MOTOR4.3
- removed net EN4_SIG: CR2.DIN, R20.1, U10.D
- removed net M_EN_0: EROW.8, R13.1, U1.PE0, U7.S
- removed net M_EN_1: EROW.7, R15.1, U1.PE1, U8.S
- removed net M_EN_2: EROW.6, R17.1, U1.PE2, U9.S
- removed net M_EN_3: EROW.5, R19.1, U1.PE3, U10.S
- removed net N$36: FROW.1
- removed net N$37: FROW.2
- removed net N$38: FROW.3
- removed net N$44: EROW.1
- removed net N$45: EROW.2
- removed net PC5: CROW.3, U1.PC5
- removed net PD4: DROW.4, U1.PD4
- removed net PF4: FROW.4, U1.PF4
- new net ENDEFF: U1.PD4
- new net PB6: U1.PB6
- new net PB7: U1.PB7
- new net PE0: U1.PE0
- new net PE1: U1.PE1
- new net PE2: U1.PE2
- new net PE3: U1.PE3
- net !DIR1: now also MOTOR1.4, MOTOR2.4; no longer MOTOR1.6
- net !DIR2: no longer MOTOR2.6
- net !DIR3: now also MOTOR3.4; no longer MOTOR3.6
- net !DIR4: now also MOTOR4.4; no longer MOTOR4.6
- net !RST: now also PROG.5
- net !RS_RX: now also RS485.2; no longer RS485OUT.4
- net !RS_TX: now also RS485.4; no longer RS485OUT.2
- net 3.3V: no longer R13.2, R15.2, R17.2, R19.2, U10.G, U7.G, U8.G, U9.G
- net 5V: now also C15.1, IC2.VCC; no longer CR2.VCC, R14.2, R16.2, R18.2, R20.2
- net DIR1: now also MOTOR1.3, MOTOR2.3; no longer MOTOR1.5
- net DIR2: no longer MOTOR2.5
- net DIR3: now also MOTOR3.3; no longer MOTOR3.5
- net DIR4: now also MOTOR4.3; no longer MOTOR4.5
- net GND: now also MOTOR1.5, MOTOR2.5, MOTOR3.5, MOTOR4.5, RS485.5; no longer C18.2, C19.2, CR2.!EN, CR2.EN, CR2.GND, IC3.GND, RS485OUT.1
- net M_DIR_0: no longer DROW.8
- net M_DIR_1: no longer DROW.7
- net M_DIR_2: no longer DROW.6
- net M_DIR_3: no longer DROW.5
- net PA2: no longer AROW.6
- net PA3: no longer AROW.5
- net PA4: no longer AROW.4
- net PA5: no longer AROW.3
- net PA6: no longer AROW.2
- net PA7: no longer AROW.1
- net PB2: no longer BROW.6
- net PB3: no longer BROW.5
- net PB4: no longer BROW.4
- net PB5: no longer BROW.3
- net PC4: no longer CROW.4
- net PC6: no longer CROW.2
- net PC7: no longer CROW.1
- net PD5: no longer DROW.3
- net PE4: no longer EROW.4
- net PE5: no longer EROW.3
- net PF0: no longer FROW.8
- net PF1: no longer FROW.7
- net RS_RX: now also RS485.1; no longer RS485OUT.5
- net RS_TX: now also RS485.3; no longer RS485OUT.3
- net T0PWM0: now also U1.PF4; no longer BROW.2, U1.PB6
- net T0PWM1: now also U1.PC5; no longer BROW.1, U1.PB7
- net T1PWM0: no longer FROW.6
- net T1PWM1: no longer FROW.5
- net TCK: now also PROG.1; no longer CROW.8
- net TDI: now also PROG.4; no longer CROW.6
- net TDO: now also PROG.3; no longer CROW.5
- net TMS: now also PROG.2; no longer CROW.7
- net U0RX: now also IC2.TXD; no longer AROW.8
- net U0TX: now also IC2.RXD; no longer AROW.7
- net U1RX: now also U2.R; no longer BROW.8, IC2.TXD
- net U1TX: now also U2.D; no longer BROW.7, IC2.RXD
- net U2RX: no longer DROW.2, U2.R
- net U2TX: no longer DROW.1, U2.D
- net V_USB: no longer C15.1, IC2.VCC
Other:
- note removed: "3.3V Linear Regulator"
- note removed: "5V Linear Regulator"
- moved on the sheet: J1, J3, J4, J7, R21, R22, R23, R24, R25, R26, R27, R28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

Commit message: new boards
Parts:
- added H1, H2, H3, H4: MOUNT-HOLE3.2, holes:MOUNT-HOLE3.2
- added J2: (no value), SparkFun-Connectors:CONN_02
- added U$1: ENDTIVA, tiva:ENDTIVA
- renumbered U2 to SN75
Connections:
- removed net EXT_DBG: J3.3
- net !DIR1: no longer MOTOR2.4
- net !DIR2: now also MOTOR2.4
- net 3.3V: now also U$1.3.3V
- net 5V: now also J2.1
- net DIR1: no longer MOTOR2.3
- net DIR2: now also MOTOR2.3
- net ENDEFF: now also U$1.DIO
- net GND: now also U$1.GND
- net U0RX: no longer J3.1
- net U0TX: no longer J3.2
- net V_USB: now also J2.2

Commit message: final board prelim final design
Parts:
- added J5: (no value), SparkFun-Connectors:CONN_02
- added U$2: BM05B-ZESS, tiva:BM05B-ZESS
Connections:
- new net 3.3VIN: 3.3V.VOUT, C17.1, IC2.3V3OUT, IC2.VCCIO, J5.2, U$2.3
- net 3.3V: now also J5.1, U$2.4; no longer 3.3V.VOUT, C17.1, IC2.3V3OUT, IC2.VCCIO
- net 5V: now also U$2.2
- net GND: now also U$2.5
- net V_USB: now also U$2.1
Changed lines of the file:
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@@
 <part name="GND19" library="SparkFun-PowerSymbols" library_urn="urn:adsk.eagle:library:530" deviceset="GND" device=""/>
 <part name="J2" library="SparkFun-Connectors" library_urn="urn:adsk.eagle:library:513" deviceset="CONN_02" device="" package3d_urn="urn:adsk.eagle:package:38039/1"/>
+<part name="U$2" library="tiva" deviceset="BM05B-ZESS" device=""/>
+<part name="J5" library="SparkFun-Connectors" library_urn="urn:adsk.eagle:library:513" deviceset="CONN_02" device="" package3d_urn="urn:adsk.eagle:package:38039/1"/>
 </parts>
 <sheets>
@@
 <attribute name="VALUE" x="68.58" y="38.354" size="1.778" layer="96" font="vector"/>
 <attribute name="NAME" x="68.58" y="48.768" size="1.778" layer="95" font="vector"/>
+</instance>
+<instance part="U$2" gate="G$1" x="109.22" y="20.32" smashed="yes">
+<attribute name="NAME" x="109.22" y="17.78" size="1.778" layer="95"/>
+<attribute name="VALUE" x="109.22" y="15.24" size="1.778" layer="96"/>
+</instance>
+<instance part="J5" gate="G$1" x="71.12" y="30.48" smashed="yes">
+<attribute name="VALUE" x="68.58" y="25.654" size="1.778" layer="96" font="vector"/>
+<attribute name="NAME" x="68.58" y="36.068" size="1.778" layer="95" font="vector"/>
 </instance>
 </instances>
@@
 </segment>
 <segment>
-<pinref part="3.3V" gate="G$1" pin="VOUT"/>
-<wire x1="132.08" y1="88.9" x2="137.16" y2="88.9" width="0.1524" layer="91"/>
-<label x="142.24" y="88.9" size="1.778" layer="95"/>
-<pinref part="C17" gate="G$1" pin="1"/>
-<wire x1="137.16" y1="88.9" x2="144.78" y2="88.9" width="0.1524" layer="91"/>
-<wire x1="137.16" y1="83.82" x2="137.16" y2="88.9" width="0.1524" layer="91"/>
-<junction x="137.16" y="88.9"/>
-</segment>
-<segment>
 <pinref part="SUPPLY7" gate="G$1" pin="3.3V"/>
 <pinref part="R2" gate="G$1" pin="2"/>
 <wire x1="177.8" y1="96.52" x2="177.8" y2="93.98" width="0.1524" layer="91"/>
+</segment>
+<segment>
+<pinref part="U$2" gate="G$1" pin="4"/>
+<wire x1="121.92" y1="27.94" x2="137.16" y2="27.94" width="0.1524" layer="91"/>
+<label x="129.54" y="27.94" size="1.778" layer="95"/>
+</segment>
+<segment>
+<pinref part="J5" gate="G$1" pin="1"/>
+<wire x1="78.74" y1="30.48" x2="88.9" y2="30.48" width="0.1524" layer="91"/>
+<label x="81.28" y="30.48" size="1.778" layer="95"/>
 </segment>
 </net>
@@
 <wire x1="177.8" y1="73.66" x2="177.8" y2="66.04" width="0.1524" layer="91"/>
 </segment>
+<segment>
+<pinref part="U$2" gate="G$1" pin="5"/>
+<wire x1="121.92" y1="22.86" x2="137.16" y2="22.86" width="0.1524" layer="91"/>
+<label x="129.54" y="22.86" size="1.778" layer="95"/>
+</segment>
 </net>
 <net name="VDDC" class="0">
@@
 <segment>
 <pinref part="J2" gate="G$1" pin="2"/>
-<wire x1="78.74" y1="45.72" x2="86.36" y2="43.18" width="0.1524" layer="91"/>
-<label x="81.28" y="43.18" size="1.778" layer="95"/>
+<wire x1="78.74" y1="45.72" x2="86.36" y2="45.72" width="0.1524" layer="91"/>
+<label x="81.28" y="45.72" size="1.778" layer="95"/>
+</segment>
+<segment>
+<pinref part="U$2" gate="G$1" pin="1"/>
+<wire x1="121.92" y1="43.18" x2="137.16" y2="43.18" width="0.1524" layer="91"/>
+<label x="129.54" y="43.18" size="1.778" layer="95"/>
 </segment>
 </net>
@@
 <segment>
 <pinref part="J2" gate="G$1" pin="1"/>
-<wire x1="78.74" y1="43.18" x2="86.36" y2="45.72" width="0.1524" layer="91"/>
-<label x="81.28" y="45.72" size="1.778" layer="95"/>
+<wire x1="78.74" y1="43.18" x2="88.9" y2="43.18" width="0.1524" layer="91"/>
+<label x="81.28" y="43.18" size="1.778" layer="95"/>
+</segment>
+<segment>
+<pinref part="U$2" gate="G$1" pin="2"/>
+<wire x1="121.92" y1="38.1" x2="137.16" y2="38.1" width="0.1524" layer="91"/>
+<label x="129.54" y="38.1" size="1.778" layer="95"/>
+</segment>
+</net>
+<net name="3.3VIN" class="0">
+<segment>
+<pinref part="3.3V" gate="G$1" pin="VOUT"/>
+<wire x1="132.08" y1="88.9" x2="137.16" y2="88.9" width="0.1524" layer="91"/>
+<label x="142.24" y="88.9" size="1.778" layer="95"/>
+<pinref part="C17" gate="G$1" pin="1"/>
+<wire x1="137.16" y1="88.9" x2="144.78" y2="88.9" width="0.1524" layer="91"/>
+<wire x1="137.16" y1="83.82" x2="137.16" y2="88.9" width="0.1524" layer="91"/>
+<junction x="137.16" y="88.9"/>
+</segment>
+<segment>
+<pinref part="U$2" gate="G$1" pin="3"/>
+<wire x1="121.92" y1="33.02" x2="137.16" y2="33.02" width="0.1524" layer="91"/>
+<label x="129.54" y="33.02" size="1.778" layer="95"/>
+</segment>
+<segment>
+<pinref part="J5" gate="G$1" pin="2"/>
+<wire x1="78.74" y1="33.02" x2="88.9" y2="33.02" width="0.1524" layer="91"/>
+<label x="81.28" y="33.02" size="1.778" layer="95"/>
 </segment>
 </net>
@@
 <nets>
 <net name="3.3V" class="0">
-<segment>
-<pinref part="IC2" gate="G$1" pin="3V3OUT"/>
-<wire x1="60.96" y1="101.6" x2="58.42" y2="101.6" width="0.1524" layer="91"/>
-<pinref part="IC2" gate="G$1" pin="VCCIO"/>
-<wire x1="58.42" y1="101.6" x2="50.8" y2="101.6" width="0.1524" layer="91"/>
-<wire x1="60.96" y1="99.06" x2="58.42" y2="99.06" width="0.1524" layer="91"/>
-<wire x1="58.42" y1="99.06" x2="58.42" y2="101.6" width="0.1524" layer="91"/>
-<junction x="58.42" y="101.6"/>
-<label x="50.8" y="101.6" size="1.778" layer="95"/>
-</segment>
 <segment>
 <wire x1="121.92" y1="137.16" x2="121.92" y2="129.54" width="0.1524" layer="91"/>
@@
 </segment>
 </net>
+<net name="3.3VIN" class="0">
+<segment>
+<pinref part="IC2" gate="G$1" pin="3V3OUT"/>
+<wire x1="60.96" y1="101.6" x2="58.42" y2="101.6" width="0.1524" layer="91"/>
+<pinref part="IC2" gate="G$1" pin="VCCIO"/>
+<wire x1="58.42" y1="101.6" x2="50.8" y2="101.6" width="0.1524" layer="91"/>
+<wire x1="60.96" y1="99.06" x2="58.42" y2="99.06" width="0.1524" layer="91"/>
+<wire x1="58.42" y1="99.06" x2="58.42" y2="101.6" width="0.1524" layer="91"/>
+<junction x="58.42" y="101.6"/>
+<label x="50.8" y="101.6" size="1.778" layer="95"/>
+</segment>
+</net>

Commit message: Fix Firmware
Parts:
- PROG: value BM05B-ZESS -> BM08B-ZESS; device tiva:BM05B-ZESS -> tiva:BM08B-ZESS
- renumbered U$1 to ENDEFFECTOR, U$2 to SWITCH
Connections:
- net !RST: now also PROG.P$4; no longer PROG.5
- net 5V: now also PROG.P$2
- net GND: now also PROG.P$1
- net TCK: now also PROG.P$8; no longer PROG.1
- net TDI: now also PROG.P$5; no longer PROG.4
- net TDO: now also PROG.P$6; no longer PROG.3
- net TMS: now also PROG.P$7; no longer PROG.2
Other:
- note removed: "check this part"
